File: PCB_design/ESP_smt_PCB/drone/drone.kicad_pcb (KiCad board)
At the start: 2 copper layers, 58 x 58 mm, 67 parts, among them J1 USB_B_Micro, J11 Conn_2, J16 Conn_2, J2 Conn_01x09, J21 Conn_2, J23 Conn_01x02_Pin, J24 Conn_01x08, J4 Conn_2, Q1 AO3400A, Q2 AO3400A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

Commit message: Holes in the pcb
Parts:
- J11, J16, J21, J4: footprint Connector_PinSocket_2.00mm:PinSocket_1x02_P2.00mm_Horizontal -> Connector_JST:JST_XH_S2B-XH-A-1_1x02_P2.50mm_Horizontal
- SW3: footprint Button_Switch_THT:SW_Tactile_SPST_Angled_PTS645Vx39-2LFS -> Button_Switch_SMD:SW_DIP_SPSTx01_Slide_6.7x4.1mm_W8.61mm_P2.54mm_LowProfile
- moved Q3 2.83 mm to (244.4, 98.4)
- moved R3 1.76 mm to (205.4, 89.2)
- moved C3 1.58 mm to (208.6, 85.5)
- moved SW3 1.47 mm to (244.1, 104.4)
- moved J1 0.46 mm to (203.4, 80.5)
- turned J11 to 90 degrees
- turned J16 to 90 degrees
- turned J21 to -90 degrees
- turned J4 to -90 degrees
Routing:
- net VDD33: track 143.8 -> 152.2 mm, vias 7 -> 6
- net VBAT: track 170.9 -> 176.3 mm, vias 2 -> 3
- net Net-(J1-D+): track 8.48 -> 4.48 mm
- net VBUS: track 93.1 -> 89.3 mm
- net ESP_EN: track 139.9 -> 136.9 mm
- net Net-(J16-Pin_1): track 4.61 -> 7.50 mm
- net VL5_SCL: track 22.1 -> 24.6 mm
- net VL5_LP: track 24.2 -> 26.1 mm
- net VL5_SDA: track 19.1 -> 20.7 mm
- net ESP_IO0: track 80.1 -> 81.4 mm
- net VDD_CP: track 20.0 -> 21.0 mm
- net MOT_3: track 50.3 -> 51.3 mm
- net Net-(J1-D-): track 5.10 -> 4.34 mm
- net VL5_RESET: track 16.2 -> 15.5 mm
- added copper zone on B.Cu, net GND
- added copper zone on F.Cu, net GND
Other:
- outline, holes or cut-outs redrawn
