File: PCB_design/ESP_plug_PCB/drone/drone.kicad_sch (KiCad schematic)
At the start: 42 parts, among them J1 Conn_02x08_Odd_Even, J11 Conn_2, J16 Conn_2, J2 Conn_01x09, J21 Conn_2, J23 Conn_01x02_Pin, J24 Conn_01x08, J4 Conn_2, J6 Conn_02x08_Odd_Even, Q1 AO3400A, Q2 AO3400A, Q3 AO3400A, Q4 AO3400A, Q6 AO3401A, U5 AP2112K-3.3TRG1, U6 MPU-6050

Commit message: fix pcb plug
Parts:
- added U1: ESP32-S3-MINI-1, symbol MCU_Espressif:ESP32-S3-MINI-1
- J1, J6: footprint Connector_PinHeader_2.54mm:PinHeader_2x08_P2.54mm_Vertical -> Connector_PinSocket_2.54mm:PinSocket_2x08_P2.54mm_Vertical
Connections:
- net ADC_BAT: now also J6.5 (Pin_5); no longer J6.6 (Pin_6)
- net BUZ_1: now also J1.12 (Pin_12); no longer J1.11 (Pin_11)
- net BUZ_2: now also J1.16 (Pin_16); no longer J1.15 (Pin_15)
- net ESP_EN: now also J6.2 (Pin_2); no longer J6.1 (Pin_1)
- net LED_B: now also J6.14 (Pin_14); no longer J6.13 (Pin_13)
- net LED_G: now also J6.12 (Pin_12); no longer J6.11 (Pin_11)
- net LED_R: now also J6.10 (Pin_10); no longer J6.9 (Pin_9)
- net MOT_1: now also J6.4 (Pin_4); no longer J6.3 (Pin_3)
- net MOT_2: now also J1.11 (Pin_11); no longer J1.12 (Pin_12)
- net MOT_3: now also J6.15 (Pin_15); no longer J6.16 (Pin_16)
- net MOT_4: now also J6.13 (Pin_13); no longer J6.14 (Pin_14)
- net MPU_INT: now also J6.7 (Pin_7); no longer J6.8 (Pin_8)
- net MPU_SCL: now also J6.6 (Pin_6); no longer J6.5 (Pin_5)
- net VBUS: now also J1.15 (Pin_15); no longer J1.16 (Pin_16)
- net VL5_INT: now also J1.1 (Pin_1); no longer J1.2 (Pin_2)
- net VL5_LP: now also J1.5 (Pin_5); no longer J1.6 (Pin_6)
- net VL5_RESET: now also J1.3 (Pin_3); no longer J1.4 (Pin_4)
- net VL5_SCL: now also J6.8 (Pin_8); no longer J6.7 (Pin_7)
- net VL5_SDA: now also J6.9 (Pin_9); no longer J6.10 (Pin_10)
- new net: U1.1 (GND), U1.2 (GND), U1.42 (GND), U1.43 (GND), U1.46 (GND), U1.47 (GND), U1.48 (GND), U1.49 (GND), U1.50 (GND), U1.51 (GND), U1.52 (GND), U1.53 (GND), U1.54 (GND), U1.55 (GND), U1.56 (GND), U1.57 (GND), U1.58 (GND), U1.59 (GND), U1.60 (GND), U1.61 (GND), U1.62 (GND), U1.63 (GND), U1.64 (GND), U1.65 (GND)
Other:
- note added: "03/05/2026"
- note added: "1.0"
- note added: "Done by Rui Bartolome - rui.bartolome@gmail.com Revised by Juan Sebastián Cely - juan.cely@urjc.es"
- note added: "ESP Soccers"
- note added: "LED"
- note added: "Micro drone PCB - plugable ESP32-S2-mini"
- note removed: "LEDs"
- note removed: "SoC"
- moved on the sheet: C6, C7, C8, C9, D5, D6, D7, D8, D9, J1, J11, J16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
