File: PCB_design/ESP_plug_PCB/drone/drone.kicad_pcb (KiCad board)
At the start: 2 copper layers, 58 x 58 mm, 67 parts, among them J1 USB_B_Micro, J11 Conn_2, J16 Conn_2, J2 Conn_01x09, J21 Conn_2, J23 Conn_01x02_Pin, J24 Conn_01x08, J4 Conn_2, Q1 AO3400A, Q2 AO3400A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

Commit message: Pcb with holes
Parts:
- removed C1, C3: 4.7uF/10V, Capacitor_SMD:C_0201_0603Metric
- removed C12, C13, C17, C2, C4, C5: 0.1uF/10V, Capacitor_SMD:C_0201_0603Metric
- removed C16: 10uF/10V, Capacitor_SMD:C_0201_0603Metric
- removed L1: BLM18SG331TN1D, Inductor_SMD:L_0201_0603Metric
- removed R1, R2: 0R/1%, Resistor_SMD:R_0201_0603Metric
- removed R12, R34, R35, R5, R6, R7: 10K/1%, Resistor_SMD:R_0201_0603Metric
- removed R3: 22.1k/1%, Resistor_SMD:R_0201_0603Metric
- removed R4: 47.5K/1%, Resistor_SMD:R_0201_0603Metric
- removed SW1: SW_Push, Button_Switch_SMD:SW_DIP_SPSTx01_Slide_6.7x4.1mm_W8.61mm_P2.54mm_LowProfile
- removed SW3: SW_Push, Button_Switch_THT:SW_Tactile_SPST_Angled_PTS645Vx39-2LFS
- removed U1: ESP32-S3-MINI-1, RF_Module:ESP32-S2-MINI-1
- removed U2: USBLC6-2SC6, Package_TO_SOT_SMD:SOT-23-6
- removed U3: CP2102N-A02-GQFN28, usb_bridge:CP2102N-A02-GQFN28
- removed U4: BC847CDW1T1G, transistor:BC847CDW1T1G
- added J3: Conn_01x08, Connector_PinHeader_2.54mm:PinHeader_1x08_P2.54mm_Vertical, F.Cu at (220.5, 71.0)
- added J5: Conn_01x08, Connector_PinHeader_2.54mm:PinHeader_1x08_P2.54mm_Vertical, F.Cu at (236.5, 53.5)
- added J6: Conn_01x08, Connector_PinHeader_2.54mm:PinHeader_1x08_P2.54mm_Vertical, F.Cu at (241.0, 71.3)
- J1: value USB_B_Micro -> Conn_01x08; footprint Connector_USB:USB_Micro-B_Amphenol_10118193-0002LF_Horizontal -> Connector_PinHeader_2.54mm:PinHeader_1x08_P2.54mm_Vertical
- J11, J16, J21, J4: footprint Connector_PinSocket_2.00mm:PinSocket_1x02_P2.00mm_Horizontal -> Connector_JST:JST_XH_S2B-XH-A-1_1x02_P2.50mm_Horizontal
- moved J1 30.9 mm to (216.9, 53.2), turned to 0 degrees
- moved R15 9.31 mm to (210.8, 63.0)
- moved R14 6.08 mm to (211.7, 65.0)
- moved J4 2.79 mm to (205.6, 59.5), turned to -90 degrees
- moved J16 2.65 mm to (252.4, 99.2), turned to 90 degrees
- moved J21 2.00 mm to (205.8, 96.8), turned to -90 degrees
- moved J11 1.48 mm to (252.3, 63.3), turned to 90 degrees
Connections:
- J1 pad 1: VBUS -> ESP_EN
- J1 pad 2: Net-(J1-D-) -> MOT_1
- J1 pad 3: Net-(J1-D+) -> MPU_SCL
- J1 pad 4: unconnected-(J1-ID-Pad4) -> VL5_SCL
- J1 pad 5: GND -> LED_R
- J1 pad 6: unconnected-(J1-Shield-Pad6)_1 -> LED_G
Routing:
- net ESP_IO0: track 80.1 -> 0.00 mm, vias 6 -> 0
- net ESP_EN: track 139.9 -> 60.7 mm, vias 6 -> 0
- net VDD33_ESP: track 50.6 -> 0.00 mm, vias 3 -> 0
- net CP_RXD: track 50.0 -> 0.00 mm, vias 2 -> 0
- net VBUS: track 93.1 -> 45.6 mm, vias 2 -> 0
- net CP_TXD: track 45.9 -> 0.00 mm, vias 2 -> 0
- net VL5_SCL: track 22.1 -> 56.9 mm, vias 0 -> 1
- net CP_RTS: track 26.0 -> 0.00 mm, vias 2 -> 0
- net CP_DTR: track 21.4 -> 0.00 mm
- net VDD33: track 143.8 -> 122.7 mm, vias 7 -> 4
- net VDD_CP: track 20.0 -> 0.00 mm, vias 2 -> 0
- net LED_G: track 22.6 -> 5.72 mm, vias 2 -> 1
- net VL5_SDA: track 19.1 -> 34.4 mm, vias 2 -> 0
- net MPU_SCL: track 20.7 -> 35.7 mm
- net MPU_SDA: track 23.0 -> 8.22 mm
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- added copper zone on B.Cu, net GND
- added copper zone on F.Cu, net GND
Other:
- outline, holes or cut-outs redrawn

Commit message: fix
Parts:
- removed J3, J5: Conn_01x08, Connector_PinHeader_2.54mm:PinHeader_1x08_P2.54mm_Vertical
- J1, J6: value Conn_01x08 -> Conn_02x08_Odd_Even; footprint Connector_PinHeader_2.54mm:PinHeader_1x08_P2.54mm_Vertical -> Connector_PinHeader_2.54mm:PinHeader_2x08_P2.54mm_Vertical
- moved J6 28.1 mm to (218.0, 55.2), turned to 0 degrees
- moved J1 21.2 mm to (238.0, 55.2)
- moved C7 4.79 mm to (224.2, 101.2), turned to 0 degrees
- moved C9 4.60 mm to (221.4, 94.5), turned to 0 degrees
- moved C6 4.37 mm to (224.2, 103.8)
- moved C8 2.69 mm to (221.8, 97.0)
- moved R18 2.54 mm to (234.8, 74.8)
- moved R10 1.99 mm to (244.4, 94.0), turned to 0 degrees
- moved R9 1.97 mm to (243.2, 56.5), turned to 180 degrees
- moved R8 1.79 mm to (214.5, 58.3)
- moved R16 1.76 mm to (234.2, 94.5)
- moved R14 1.55 mm to (213.2, 64.8)
- moved Q2 1.49 mm to (246.8, 56.7), turned to -90 degrees
- moved C10 1.36 mm to (226.3, 77.0)
Connections:
- J1 pad 1: ESP_EN -> unconnected-(J1-Pin_1-Pad1)
- J1 pad 2: MOT_1 -> VL5_INT
- J1 pad 3: MPU_SCL -> unconnected-(J1-Pin_3-Pad3)
- J1 pad 4: VL5_SCL -> VL5_RESET
- J1 pad 5: LED_R -> unconnected-(J1-Pin_5-Pad5)
- J1 pad 6: LED_G -> VL5_LP
- J1 pad 7: LED_B -> unconnected-(J1-Pin_7-Pad7)
- J1 pad 8: VDD33 -> unconnected-(J1-Pin_8-Pad8)
- J6 pad 1: VBUS -> ESP_EN
- J6 pad 2: GND -> unconnected-(J6-Pin_2-Pad2)
- J6 pad 3: MOT_2 -> MOT_1
- J6 pad 5: unconnected-(J6-Pin_5-Pad5) -> MPU_SCL
- J6 pad 6: VL5_LP -> ADC_BAT
- J6 pad 7: VL5_RESET -> VL5_SCL
- J6 pad 8: VL5_INT -> MPU_INT
Routing:
- net GND: track 0.00 -> 101.8 mm, vias 0 -> 13
- net LED_G: track 5.72 -> 16.6 mm
- net BUZ_1: track 25.4 -> 19.1 mm
- net VL5_SCL: track 56.9 -> 51.2 mm
- net VBAT: track 171.5 -> 176.2 mm
- net MOT_2: track 13.6 -> 18.2 mm
- net VSYS: track 59.8 -> 64.4 mm
- net MPU_INT: track 25.3 -> 21.2 mm
- net VL5_INT: track 21.6 -> 25.6 mm
- net MPU_SCL: track 35.7 -> 32.9 mm
- net VBUS: track 45.6 -> 42.8 mm
- net MOT_4: track 40.9 -> 38.3 mm
- net VDD33: track 122.7 -> 125.1 mm
- net ESP_EN: track 60.7 -> 58.3 mm, vias 0 -> 2
- net BUZ_2: track 17.5 -> 15.2 mm
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
Commit message: Fix 3.3v
Parts:
- moved R18 0.95 mm to (234.8, 73.8)
Connections:
- J6 pad 15: VDD33 -> unconnected-(J6-Pin_15-Pad15)
Routing:
- net VDD33: track 125.1 -> 98.3 mm
- net GND: track 101.8 -> 91.3 mm, vias 13 -> 12

Commit message: fix pcb plug
Parts:
- added U1: ESP32-S3-MINI-1, RF_Module:ESP32-S2-MINI-1, F.Cu at (229.8, 64.8)
- J1, J6: footprint Connector_PinHeader_2.54mm:PinHeader_2x08_P2.54mm_Vertical -> Connector_PinSocket_2.54mm:PinSocket_2x08_P2.54mm_Vertical
- moved C10 2.79 mm to (223.6, 76.4), turned to -90 degrees
- moved U6 2.69 mm to (229.0, 78.6)
- moved J1 2.65 mm to (240.5, 55.8)
- moved R19 2.36 mm to (233.7, 81.6), turned to 180 degrees
- moved R20 2.34 mm to (233.7, 80.2), turned to 180 degrees
- moved J6 2.22 mm to (220.1, 55.8)
- moved C11 1.08 mm to (234.3, 77.8)
Connections:
- J1 pad 1: unconnected-(J1-Pin_1-Pad1) -> VL5_INT
- J1 pad 11: BUZ_1 -> MOT_2
- J1 pad 12: MOT_2 -> BUZ_1
- J1 pad 15: BUZ_2 -> VBUS
- J1 pad 16: VBUS -> BUZ_2
- J1 pad 2: VL5_INT -> unconnected-(J1-Pin_2-Pad2)
- J1 pad 3: unconnected-(J1-Pin_3-Pad3) -> VL5_RESET
- J1 pad 4: VL5_RESET -> unconnected-(J1-Pin_4-Pad4)
- J1 pad 5: unconnected-(J1-Pin_5-Pad5) -> VL5_LP
- J1 pad 6: VL5_LP -> unconnected-(J1-Pin_6-Pad6)
- J6 pad 1: ESP_EN -> unconnected-(J6-Pin_1-Pad1)
- J6 pad 10: VL5_SDA -> LED_R
- J6 pad 11: LED_G -> unconnected-(J6-Pin_11-Pad11)
- J6 pad 12: unconnected-(J6-Pin_12-Pad12) -> LED_G
- J6 pad 13: LED_B -> MOT_4
- J6 pad 14: MOT_4 -> LED_B
- J6 pad 15: unconnected-(J6-Pin_15-Pad15) -> MOT_3
- J6 pad 16: MOT_3 -> unconnected-(J6-Pin_16-Pad16)
- J6 pad 2: unconnected-(J6-Pin_2-Pad2) -> ESP_EN
- J6 pad 3: MOT_1 -> unconnected-(J6-Pin_3-Pad3)
- J6 pad 4: unconnected-(J6-Pin_4-Pad4) -> MOT_1
- J6 pad 5: MPU_SCL -> ADC_BAT
- J6 pad 6: ADC_BAT -> MPU_SCL
- J6 pad 7: VL5_SCL -> MPU_INT
- J6 pad 8: MPU_INT -> VL5_SCL
- J6 pad 9: LED_R -> VL5_SDA
Routing:
- net VDD33: track 98.3 -> 104.1 mm
- net MOT_3: track 43.6 -> 48.4 mm, vias 2 -> 1
- net GND: track 91.3 -> 95.5 mm
- net MPU_SDA: track 8.22 -> 5.08 mm
- net AUX_SDA: track 8.78 -> 6.28 mm
- net Net-(U6-REGOUT): track 1.50 -> 3.24 mm
- net MPU_INT: track 21.6 -> 23.3 mm
- net Net-(U6-CPOUT): track 2.96 -> 3.92 mm
- net BUZ_2: track 15.2 -> 14.3 mm
- net MPU_SCL: track 33.3 -> 34.0 mm, vias 2 -> 0
- net BUZ_1: track 19.1 -> 18.5 mm
- net ESP_EN: track 58.3 -> 58.9 mm
- net MOT_2: track 18.2 -> 18.8 mm
- net AUX_SCL: track 8.04 -> 7.67 mm, vias 2 -> 1
