File: PCB_design/ESP_plug_mini_PCB/drone/drone.kicad_pcb (KiCad board)
At the start: 2 copper layers, 39.9 x 39.7 mm, 39 parts, among them J1 Conn_02x08_Odd_Even, J11 Conn_2, J16 Conn_2, J21 Conn_2, J23 Conn_01x02_Pin, J4 Conn_2, J6 Conn_02x08_Odd_Even, Q1 AO3400A, Q2 AO3400A, Q3 AO3400A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

Commit message: pcb updated
Parts:
- J11, J16, J21, J4: moved to B.Cu
- moved Q2 134.9 mm to (233.3, 90.8)
- moved R9 134.9 mm to (230.3, 90.8)
- moved J16 127.7 mm to (234.5, 116.2), turned to -135 degrees
- moved C7 127.6 mm to (220.6, 109.8), turned to 180 degrees
- moved J21 127.1 mm to (199.7, 117.8), turned to 135 degrees
- moved R14 125.8 mm to (200.9, 97.2)
- moved R15 125.8 mm to (198.7, 97.0)
- moved D7 125.7 mm to (197.5, 98.9)
- moved D8 125.7 mm to (197.5, 100.8)
- moved D6 125.6 mm to (197.4, 104.8)
- moved D9 125.6 mm to (197.4, 102.8)
- moved C10 125.6 mm to (210.8, 98.3)
- moved C6 125.3 mm to (211.8, 114.2)
- moved R16 125.3 mm to (216.1, 108.9)
- moved C11 125.3 mm to (220.4, 98.5)
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Routing:
- net GND: track 6.13 -> 46.3 mm, vias 0 -> 8
- net VDD33: track 41.6 -> 60.0 mm, vias 1 -> 2
- net VBAT: track 115.2 -> 129.4 mm
- net MOT_2: track 28.0 -> 14.3 mm
- net Net-(J4-Pin_1): track 6.57 -> 8.58 mm
- net MOT_4: track 9.44 -> 11.3 mm
- net VSYS: track 34.1 -> 35.8 mm
- net ADC_BAT: track 10.5 -> 12.2 mm
- net Net-(J21-Pin_2): track 6.35 -> 5.07 mm
- net MOT_1: track 12.0 -> 11.0 mm
- net Net-(J11-Pin_2): track 6.74 -> 7.75 mm
- net Net-(U6-CPOUT): track 2.74 -> 2.18 mm
- net AUX_SCL: vias 1 -> 0
Other:
- board size 39.9 x 39.7 mm -> 90.9 x 90.6 mm
- board text added: "Conn_2"
- board text removed: "J21"
