File: PCB_design/ESP_plug_mini_PCB_gy87/drone/drone.kicad_pcb (KiCad board)
At the start: 2 copper layers, 91.5 x 91.4 mm, 34 parts, among them J1 Conn_02x08_Odd_Even, J11 Conn_2, J16 Conn_2, J2 Conn_01x08, J21 Conn_2, J23 Conn_01x02_Pin, J4 Conn_2, J6 Conn_02x08_Odd_Even, Q1 AO3400A, Q2 AO3400A, Q3 AO3400A, Q4 AO3400A, U1 ESP32-S3-MINI-1, U5 AP2112K-3.3TRG1

Commit message: fixes
Parts:
- added R1: 10K/5%, Resistor_SMD:R_0201_0603Metric, F.Cu at (123.3, 96.5)
- added SW1: SW_Push, Button_Switch_SMD:SW_SPST_B3U-1000P, F.Cu at (122.5, 101.5)
- C6, C7, C8: footprint Capacitor_SMD:C_0201_0603Metric -> Capacitor_SMD:C_0603_1608Metric
- R14: footprint Resistor_SMD:R_0201_0603Metric -> Resistor_SMD:R_0402_1005Metric
- R15, R16: footprint Resistor_SMD:R_0201_0603Metric -> Resistor_SMD:R_0603_1608Metric
- R21: value 1.5K/1% -> 150/1%
- R22: value 1.5K/1% -> 270/1%
- R23: value 1.5K/1% -> 82/1%
- R24: value 1.5K/1% -> 68/1%
- moved C6 1.41 mm to (88.0, 107.2)
- moved C8 1.35 mm to (98.5, 97.8)
- moved C7 1.30 mm to (89.5, 107.2)
- moved R10 0.60 mm to (96.2, 110.8)
- moved R15 0.38 mm to (85.0, 88.0)
- moved R16 0.36 mm to (91.8, 106.5)
- moved R14 0.30 mm to (87.5, 87.5)
Connections:
- J1 pad 8: unconnected-(J1-Pin_8-Pad8) -> button
- J6 pad 15: unconnected-(J6-Pin_15-Pad15) -> MOT_3
- J6 pad 16: MOT_3 -> unconnected-(J6-Pin_16-Pad16)
Routing:
- net VDD33: track 47.4 -> 69.9 mm, vias 1 -> 3
- net button: track 0.00 -> 21.8 mm
- net VSYS: track 57.3 -> 58.3 mm
- net VBAT: track 127.7 -> 128.5 mm
