File: PCB_design/ESP_plug_mini_PCB_gy87/drone/drone.kicad_sch (KiCad schematic)
At the start: 34 parts, among them J1 Conn_02x08_Odd_Even, J11 Conn_2, J16 Conn_2, J2 Conn_01x08, J21 Conn_2, J23 Conn_01x02_Pin, J4 Conn_2, J6 Conn_02x08_Odd_Even, Q1 AO3400A, Q2 AO3400A, Q3 AO3400A, Q4 AO3400A, U1 ESP32-S3-MINI-1, U5 AP2112K-3.3TRG1

Commit message: fixes
Parts:
- added R1: 10K/5%, Resistor_SMD:R_0201_0603Metric, symbol Device:R_US
- added SW1: SW_Push, Button_Switch_SMD:SW_SPST_B3U-1000P, symbol Switch:SW_Push
- C6, C7, C8: footprint Capacitor_SMD:C_0201_0603Metric -> Capacitor_SMD:C_0603_1608Metric
- R14: footprint Resistor_SMD:R_0201_0603Metric -> Resistor_SMD:R_0402_1005Metric
- R15, R16: footprint Resistor_SMD:R_0201_0603Metric -> Resistor_SMD:R_0603_1608Metric
- R21: value 1.5K/1% -> 150/1%
- R22: value 1.5K/1% -> 270/1%
- R23: value 1.5K/1% -> 82/1%
- R24: value 1.5K/1% -> 68/1%
Connections:
- net GND: now also R1.2
- net MOT_3: now also J6.15 (Pin_15); no longer J6.16 (Pin_16)
- net VDD33: now also SW1.1
- net button: now reaches J1.8 (Pin_8)
- net button: now also R1.1, SW1.2
- no-connect marks 22 -> 21
Other:
- note added: "Button"
- note added: "GY-87 Pin Connector"
- moved on the sheet: C6, C7, C8, C9, D1, D6, D7, D8, D9, J1, J2, J23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
